File: hw/sch_pcb/4XLTO1865V02A.kicad_pcb (KiCad board)
At the start: 2 copper layers, 60.5 x 49.7 mm, 6 parts, among them J2 HEADER_2x04_PARALLEL, J3 HEADER_2x04_PARALLEL, M1 HOLE, M2 HOLE, M3 HOLE, M4 HOLE

Commit message: Edit PCB
Parts:
- moved M1 2.72 mm to (156.3, 104.1)
- moved M2 2.21 mm to (133.3, 104.1)
- moved M3 2.02 mm to (156.3, 81.1)
- moved M4 1.25 mm to (133.3, 81.1)
Changed lines of the file:
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@@
   )
   (footprint "Mlab_Mechanical:dira_19,2mm" (layer "F.Cu")
-    (at 134.232 102.108)
+    (at 133.28 104.102)
     (property "Sheetfile" "4XLTO1865V02A.kicad_sch")
     (property "Sheetname" "")
@@
   )
   (footprint "Mlab_Mechanical:dira_19,2mm" (layer "F.Cu")
-    (at 154.432 102.108)
+    (at 156.28 104.102)
     (property "Sheetfile" "4XLTO1865V02A.kicad_sch")
     (property "Sheetname" "")
@@
   )
   (footprint "Mlab_Mechanical:dira_19,2mm" (layer "F.Cu")
-    (at 134.232 81.908)
+    (at 133.28 81.102)
     (property "Sheetfile" "4XLTO1865V02A.kicad_sch")
     (property "Sheetname" "")
@@
   )
   (footprint "Mlab_Mechanical:dira_19,2mm" (layer "F.Cu")
-    (at 154.432 81.908)
+    (at 156.28 81.102)
     (property "Sheetfile" "4XLTO1865V02A.kicad_sch")
     (property "Sheetname" "")
