File: hw/sch_pcb/4XLTO1865V02A.kicad_pcb (KiCad board)
At the start: 2 copper layers, 60.5 x 49.7 mm, 6 parts, among them J2 HEADER_2x04_PARALLEL, J3 HEADER_2x04_PARALLEL, M1 HOLE, M2 HOLE, M3 HOLE, M4 HOLE

Commit message: Edit PCB
Parts:
- added M5: HOLE, Mlab_Mechanical:MountingHole_3mm, F.Cu at (119.4, 92.5)
- added M6: HOLE, Mlab_Mechanical:MountingHole_3mm, F.Cu at (170.2, 92.5)
Changed lines of the file:
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@@
     )
     (pad_to_mask_clearance 0.2)
-    (solder_mask_min_width 0.2)
     (aux_axis_origin 114.3 117.602)
     (pcbplotparams
@@
     (pad "" np_thru_hole circle (at 0 0) (size 19.2 19.2) (drill 19.2) (layers *.Mask))
   )
+  (footprint "Mlab_Mechanical:MountingHole_3mm" placed (layer "F.Cu")
+    (at 170.18 92.475)
+    (descr "Mounting hole, Befestigungsbohrung, 3mm, No Annular, Kein Restring,")
+    (tags "Mounting hole, Befestigungsbohrung, 3mm, No Annular, Kein Restring,")
+    (property "Sheetfile" "4XLTO1865V02A.kicad_sch")
+    (property "Sheetname" "")
+    (attr through_hole)
+    (fp_text reference "M6" (at 0 -4.191) (layer "F.SilkS") hide
+      (effects (font (size 1.524 1.524) (thickness 0.3048)))
+    )
+    (fp_text value "HOLE" (at 0 4.191) (layer "F.SilkS") hide
+      (effects (font (size 1.524 1.524) (thickness 0.3048)))
+    )
+    (fp_circle (center 0 0) (end 2.99974 0) (layer "F.Fab") (width 0.381) (fill none))
+    (pad "1" thru_hole circle (at 0 0) (size 6 6) (drill 3) (layers *.Cu *.Mask)
+      (net 1 "GND") (pintype "input") (clearance 1) (zone_connect 2))
+    (model "${MLAB}/src/3d/mechanical/m3_komplet.step"
+      (offset (xyz 0 0 0))
+      (scale (xyz 1 1 1))
+      (rotate (xyz 0 0 0))
+    )
+  )
+  (footprint "Mlab_Mechanical:MountingHole_3mm" placed (layer "F.Cu")
+    (at 119.38 92.475)
+    (descr "Mounting hole, Befestigungsbohrung, 3mm, No Annular, Kein Restring,")
+    (tags "Mounting hole, Befestigungsbohrung, 3mm, No Annular, Kein Restring,")
+    (property "Sheetfile" "4XLTO1865V02A.kicad_sch")
+    (property "Sheetname" "")
+    (attr through_hole)
+    (fp_text reference "M5" (at 0 -4.191) (layer "F.SilkS") hide
+      (effects (font (size 1.524 1.524) (thickness 0.3048)))
+    )
+    (fp_text value "HOLE" (at 0 4.191) (layer "F.SilkS") hide
+      (effects (font (size 1.524 1.524) (thickness 0.3048)))
+    )
+    (fp_circle (center 0 0) (end 2.99974 0) (layer "F.Fab") (width 0.381) (fill none))
+    (pad "1" thru_hole circle (at 0 0) (size 6 6) (drill 3) (layers *.Cu *.Mask)
+      (net 1 "GND") (pintype "input") (clearance 1) (zone_connect 2))
+    (model "${MLAB}/src/3d/mechanical/m3_komplet.step"
+      (offset (xyz 0 0 0))
+      (scale (xyz 1 1 1))
+      (rotate (xyz 0 0 0))
+    )
+  )
   (footprint "Mlab_Mechanical:dira_19,2mm" (layer "F.Cu")
     (at 133.28 81.102)
@@
   (gr_arc (start 114.554 77.602) (mid 117.482932 70.530932) (end 124.554 67.602) (layer "Edge.Cuts") (width 0.1))
   (gr_line (start 114.554 117.348) (end 175.006 117.348) (layer "Edge.Cuts") (width 0.1))
-  (gr_text "MLAB.CZ\n2022" (at 119.634 92.456 90) (layer "F.SilkS")
+  (gr_text "MLAB.CZ\n2022" (at 119.38 81.026 90) (layer "F.SilkS")
     (effects (font (size 1.5 1.5) (thickness 0.3)))
   )
-  (gr_text "4XLTO1865V02A\nJACHO" (at 169.672 92.202 90) (layer "F.SilkS")
+  (gr_text "4XLTO1865V02A\nJACHO" (at 170.18 78.994 90) (layer "F.SilkS")
     (effects (font (size 1.5 1.5) (thickness 0.3)))
   )
