File: hw/sch_pcb/4XLTO1865V02A.kicad_sch (KiCad schematic)
At the start: 6 parts, among them J2 HEADER_2x04_PARALLEL, J3 HEADER_2x04_PARALLEL, M1 HOLE, M2 HOLE, M3 HOLE, M4 HOLE

Commit message: Edit PCB
Parts:
- added M5, M6: HOLE, Mlab_Mechanical:MountingHole_3mm, symbol MLAB_MECHANICAL:HOLE
Connections:
- net GND: now also M5.1, M6.1
Changed lines of the file:
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@@
+    (stroke (width 0) (type default) (color 0 0 0 0))
+  )
+  (wire (pts (xy 24.13 30.48) (xy 24.13 31.115))
     (stroke (width 0) (type default) (color 0 0 0 0))
   )
@@
   )
   (wire (pts (xy 243.205 17.78) (xy 243.205 20.32))
+    (stroke (width 0) (type default) (color 0 0 0 0))
+  )
+  (wire (pts (xy 19.685 30.48) (xy 24.13 30.48))
+    (stroke (width 0) (type default) (color 0 0 0 0))
+  )
+  (wire (pts (xy 19.685 20.955) (xy 24.13 20.955))
+    (stroke (width 0) (type default) (color 0 0 0 0))
+  )
+  (wire (pts (xy 24.13 20.955) (xy 24.13 21.59))
     (stroke (width 0) (type default) (color 0 0 0 0))
   )
@@
     )
     (property "Datasheet" "" (id 3) (at 243.205 27.305 0)
+      (effects (font (size 1.27 1.27)) hide)
+    )
+    (pin "1")
+  )
+  (symbol (lib_id "power:GND") (at 24.13 21.59 0) (unit 1)
+    (in_bom yes) (on_board yes) (fields_autoplaced)
+    (property "Reference" "#PWR0103" (id 0) (at 24.13 27.94 0)
+      (effects (font (size 1.27 1.27)) hide)
+    )
+    (property "Value" "GND" (id 1) (at 24.13 26.1525 0))
+    (property "Footprint" "" (id 2) (at 24.13 21.59 0)
+      (effects (font (size 1.27 1.27)) hide)
+    )
+    (property "Datasheet" "" (id 3) (at 24.13 21.59 0)
       (effects (font (size 1.27 1.27)) hide)
     )
@@
     )
   )
+  (symbol (lib_id "MLAB_MECHANICAL:HOLE") (at 18.415 20.955 0) (unit 1)
+    (in_bom yes) (on_board yes) (fields_autoplaced)
+    (property "Reference" "M5" (id 0) (at 18.415 15.7891 0)
+      (effects (font (size 1.524 1.524)))
+    )
+    (property "Value" "HOLE" (id 1) (at 18.415 19.0681 0)
+      (effects (font (size 1.524 1.524)))
+    )
+    (property "Footprint" "Mlab_Mechanical:MountingHole_3mm" (id 2) (at 18.415 20.955 0)
+      (effects (font (size 1.524 1.524)) hide)
+    )
+    (property "Datasheet" "" (id 3) (at 18.415 20.955 0)
+      (effects (font (size 1.524 1.524)))
+    )
+    (pin "1")
+  )
+  (symbol (lib_id "MLAB_MECHANICAL:HOLE") (at 18.415 30.48 0) (unit 1)
+    (in_bom yes) (on_board yes) (fields_autoplaced)
+    (property "Reference" "M6" (id 0) (at 18.415 25.3141 0)
+      (effects (font (size 1.524 1.524)))
+    )
+    (property "Value" "HOLE" (id 1) (at 18.415 28.5931 0)
+      (effects (font (size 1.524 1.524)))
+    )
+    (property "Footprint" "Mlab_Mechanical:MountingHole_3mm" (id 2) (at 18.415 30.48 0)
+      (effects (font (size 1.524 1.524)) hide)
+    )
+    (property "Datasheet" "" (id 3) (at 18.415 30.48 0)
+      (effects (font (size 1.524 1.524)))
+    )
+    (pin "1")
+  )
   (symbol (lib_id "MLAB_MECHANICAL:HOLE_TF") (at 138.43 107.95 0) (unit 1)
     (in_bom no) (on_board yes) (fields_autoplaced)
@@
       (effects (font (size 1.524 1.524)))
     )
+  )
+  (symbol (lib_id "power:GND") (at 24.13 31.115 0) (unit 1)
+    (in_bom yes) (on_board yes) (fields_autoplaced)
+    (property "Reference" "#PWR0104" (id 0) (at 24.13 37.465 0)
+      (effects (font (size 1.27 1.27)) hide)
+    )
+    (property "Value" "GND" (id 1) (at 24.13 35.6775 0))
+    (property "Footprint" "" (id 2) (at 24.13 31.115 0)
+      (effects (font (size 1.27 1.27)) hide)
+    )
+    (property "Datasheet" "" (id 3) (at 24.13 31.115 0)
+      (effects (font (size 1.27 1.27)) hide)
+    )
+    (pin "1")
   )
   (symbol (lib_id "MLAB_HEADER:HEADER_1x04") (at 250.19 40.64 0) (unit 1)
@@
       (reference "#PWR0102") (unit 1) (value "GND") (footprint "")
     )
+    (path "/3326423d-8df7-4a7e-a354-349430b8fbd7"
+      (reference "#PWR0103") (unit 1) (value "GND") (footprint "")
+    )
+    (path "/ae77c3c8-1144-468e-ad5b-a0b4090735bd"
+      (reference "#PWR0104") (unit 1) (value "GND") (footprint "")
+    )
     (path "/7d24f687-79aa-4b8c-8284-b78868812a22"
       (reference "J2") (unit 1) (value "HEADER_2x04_PARALLEL") (footprint "Mlab_Pin_Headers:Angled_1x04")
@@
       (reference "M4") (unit 1) (value "HOLE") (footprint "Mlab_Mechanical:dira_19,2mm")
     )
-  )
+    (path "/98b00c9d-9188-4bce-aa70-92d12dd9cf82"
+      (reference "M5") (unit 1) (value "HOLE") (footprint "Mlab_Mechanical:MountingHole_3mm")
+    )
+    (path "/99332785-d9f1-4363-9377-26ddc18e6d2c"
+      (reference "M6") (unit 1) (value "HOLE") (footprint "Mlab_Mechanical:MountingHole_3mm")
+    )
+  )
